Commit message: clicked point working

File: rotors_simulator/rotors_description/urdf/multirotor_base.xacro (robot description, xacro)
@@ -57,5 +57,5 @@
         </geometry>
       </visual>
-      <collision>
+      <collision name="bump_sensor_collision">
         <origin xyz="0 0 0" rpy="0 0 0" />
         <geometry>
@@ -64,4 +64,18 @@
       </collision>
     </link>
+   <gazebo reference="${robot_namespace}/base_link">
+<maxContacts>1</maxContacts>
+   <sensor name='body_contact' type='contact'>
+          <contact>
+            <collision>firefly/base_link_fixed_joint_lump__bump_sensor_collision_collision</collision>
+	   <topic>__default_topic__</topic>
+          </contact>
+   <plugin name="body_plugin" filename="libgazebo_ros_bumper.so">
+     	<alwaysOn>true</alwaysOn>
+         <bumperTopicName>body_contact</bumperTopicName>
+         <frameName>base_link</frameName>
+   </plugin>
+   </sensor>
+   </gazebo>
     <!-- attach multirotor_base_plugin to the base_link -->
     <gazebo>
