Commit message: working, collision, sensor noise, testing

File: rotors_simulator/rotors_description/urdf/component_snippets.xacro (robot description, xacro)
@@ -363,4 +363,5 @@
         <transformTopic>${transform_topic}</transformTopic>
         <odometryTopic>${odometry_topic}</odometryTopic>
+	<suffix>${odometry_sensor_suffix}</suffix>
         <parentFrameId>${parent_frame_id}</parentFrameId> <!-- Use the scoped link name here. e.g. Model::link. -->
         <childFrameId>${child_frame_id}</childFrameId>
@@ -708,7 +709,6 @@
       </xacro:vi_sensor_depth_macro>
     </xacro:if>
-    <!-- Groundtruth -->
+    <!-- Groundtruth
     <xacro:if value="${enable_ground_truth}">
-      <!-- Odometry Sensor -->
       <xacro:odometry_plugin_macro
         namespace="${namespace}/ground_truth"
@@ -737,8 +737,8 @@
         odometry_map=""
         image_scale="">
-        <inertia ixx="0.00001" ixy="0.0" ixz="0.0" iyy="0.00001" iyz="0.0" izz="0.00001" /> <!-- [kg m^2] [kg m^2] [kg m^2] [kg m^2] [kg m^2] [kg m^2] -->
+        <inertia ixx="0.00001" ixy="0.0" ixz="0.0" iyy="0.00001" iyz="0.0" izz="0.00001" />
         <origin xyz="0.0 0.0 0.0" rpy="0.0 0.0 0.0" />
       </xacro:odometry_plugin_macro>
-    </xacro:if>
+    </xacro:if>--><!-- Odometry Sensor -->
     <!-- ADIS16448 IMU. -->
     <xacro:imu_plugin_macro
@@ -806,7 +806,7 @@
       odometry_map=""
       image_scale="">
-      <inertia ixx="0.00001" ixy="0.0" ixz="0.0" iyy="0.00001" iyz="0.0" izz="0.00001" /> <!-- [kg m^2] [kg m^2] [kg m^2] [kg m^2] [kg m^2] [kg m^2] -->
+      <inertia ixx="0.00001" ixy="0.0" ixz="0.0" iyy="0.00001" iyz="0.0" izz="0.00001" />
       <origin xyz="0.0 0.0 0.0" rpy="0.0 0.0 0.0" />
-    </xacro:odometry_plugin_macro>
+    </xacro:odometry_plugin_macro> <!-- [kg m^2] [kg m^2] [kg m^2] [kg m^2] [kg m^2] [kg m^2] -->
   </xacro:macro>
   <xacro:macro name="default_imu" params="namespace parent_link">

File: rotors_simulator/rotors_description/urdf/multirotor_base.xacro (robot description, xacro)
@@ -34,5 +34,12 @@
   <xacro:macro name="multirotor_base_macro"
     params="robot_namespace mass body_width body_height use_mesh_file mesh_file *inertia">
-    <link name="${robot_namespace}/base_link"></link>
+    <link name="${robot_namespace}/base_link">
+      <collision name="bump_sensor_collision">
+        <origin xyz="0 0 0" rpy="0 0 0" />
+        <geometry>
+          <box size="0.65 0.65 0.5" /> <!-- [m] [m] [m] -->
+        </geometry>
+      </collision>
+</link>
     <joint name="${robot_namespace}/base_joint" type="fixed">
       <origin xyz="0 0 0" rpy="0 0 0" />
@@ -57,5 +64,5 @@
         </geometry>
       </visual>
-      <collision name="bump_sensor_collision">
+      <collision>
         <origin xyz="0 0 0" rpy="0 0 0" />
         <geometry>
